File: pandashield3/newer/pandashield12-lga.brd (EAGLE design)
At the start: 114.3 x 101.7 mm, 347 parts, among them IC1 TPS773, IC2 VNH2SP30TR-E, IC3 MAX803T, IC6 VNH2SP30TR-E, IC8 LM2936MP-3.3, J1 XF2J-3024-11, J4 XF2L-0625-1, J5 XF2L-0625-1, Q2 IRLML6401, Q4 IRLML6401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

Commit message: new version of board
Parts:
- moved PAD16 13.5 mm to (11.0, 16.5)
- moved TP55 7.14 mm to (20.4, 35.6)
- moved PAD17 3.42 mm to (3.97, 14.0)
- moved PAD24 0.40 mm to (19.8, 27.4)
- moved R53 0.23 mm to (49.4, 54.6), flipped to the top, turned to 270 degrees
- flipped Q5 to the top
Routing:
- net CS_LCD: track 0.00 -> 44.1 mm, vias 0 -> 1
- net TX6: track 13.8 -> 26.0 mm
- net CS6: track 14.7 -> 26.9 mm
- net CLK6: track 14.1 -> 25.0 mm
- net RX6: track 16.1 -> 25.9 mm
- net +5V_PANDA: track 23.0 -> 30.8 mm
- net +3V3: track 127.9 -> 134.4 mm
- net VBAT: track 119.1 -> 125.0 mm, vias 9 -> 12
- net CHARGE: track 59.5 -> 65.2 mm, vias 5 -> 6
- net RX7: track 61.6 -> 66.4 mm
- net JOY_DOWN: track 99.4 -> 102.5 mm
- net MELEXIS_EN: track 71.6 -> 74.5 mm, vias 4 -> 2
- net JOY_CENT: track 101.4 -> 99.1 mm
- net JOY_LEFT: track 107.4 -> 105.5 mm
- net TX7: track 17.4 -> 19.4 mm
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- removed copper zone on layer 1, net GND
Other:
- board size 114.3 x 101.7 mm -> 114.3 x 101.9 mm

Commit message: new version in
Parts:
- removed U$100: 3,3uH, 5A, EPCOS B82464G4332M , Farnell 7429410, SparkFun:CR54
- added L1: (no value), SparkFun:CR75
- moved TP52 21.9 mm to (68.1, 41.8)
- moved C9 19.9 mm to (20.4, 34.4), turned to 180 degrees
- moved PAD24 18.1 mm to (23.2, 9.60)
- moved TP55 16.8 mm to (18.4, 18.9)
- moved C22 15.4 mm to (6.40, 39.5), turned to 90 degrees
- moved 10UF/16V 13.3 mm to (2.60, 33.4), flipped to the bottom, turned to 270 degrees
- moved C29 13.2 mm to (20.0, 31.2), turned to 180 degrees
- moved C100 13.1 mm to (8.40, 14.8), flipped to the bottom, turned to 180 degrees
- moved R11 11.6 mm to (7.97, 26.3), turned to 90 degrees
- moved R50 10.1 mm to (18.3, 41.4), turned to 90 degrees
- moved LED5 7.39 mm to (47.0, 46.8), turned to 180 degrees
- moved D100 7.25 mm to (11.1, 26.3)
- moved C33 7.07 mm to (8.40, 18.6)
- moved PAD16 6.43 mm to (11.6, 22.9)
- moved R42 6.09 mm to (47.0, 47.0), turned to 270 degrees
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Connections:
- net +5V_PANDA: now also L1.P$2; no longer U$100.P$2
- net N$33: now also L1.P$1; no longer U$100.P$1
Routing:
- net GND: track 301.7 -> 250.0 mm, vias 45 -> 51
- net +3V3: track 134.4 -> 107.1 mm, vias 21 -> 22
- net N$75: track 39.3 -> 27.1 mm
- net AN3: track 21.8 -> 10.8 mm
- net CLK0: track 41.4 -> 49.6 mm
- net LEFT_PWM: track 21.7 -> 29.0 mm
- net MOTOR1L: track 16.1 -> 10.0 mm
- net N$18: track 16.4 -> 10.3 mm, vias 0 -> 2
- net RIGHT_INB: track 56.2 -> 50.2 mm
- net +5V_PANDA: track 30.8 -> 36.8 mm, vias 2 -> 1
- net CLK2: track 94.1 -> 88.6 mm
- net CS_LCD: track 44.1 -> 38.7 mm
- net E8_TX: track 22.6 -> 28.0 mm
- net MOTOR1R: track 15.0 -> 9.74 mm
- net RX2: track 93.4 -> 88.2 mm
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Other:
- board size 114.3 x 101.9 mm -> 114.3 x 101.7 mm
