File: pandashield3/newer/pandashield12-lga.sch (EAGLE design)
At the start: 347 parts, among them IC1 TPS773, IC2 VNH2SP30TR-E, IC3 MAX803T, IC6 VNH2SP30TR-E, IC8 LM2936MP-3.3, J1 XF2J-3024-11, J4 XF2L-0625-1, J5 XF2L-0625-1, Q2 IRLML6401, Q4 IRLML6401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

Commit message: new version in
Parts:
- removed U$100: 3,3uH, 5A, EPCOS B82464G4332M , Farnell 7429410, SparkFun:INDUCTORCR54
- added L1: (no value), SparkFun:INDUCTORCR75
Connections:
- net +5V_PANDA: now also L1.2; no longer U$100.2
- net N$33: now also L1.1; no longer U$100.1
Changed lines of the file:
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@@
 <part name="GND58" library="SparkFun" deviceset="GND" device=""/>
 <part name="GND59" library="SparkFun" deviceset="GND" device=""/>
-<part name="U$100" library="SparkFun" deviceset="INDUCTOR" device="CR54" value="3,3uH, 5A, EPCOS B82464G4332M , Farnell 7429410"/>
 <part name="D100" library="diode" deviceset="BAT54" device=""/>
 <part name="GND60" library="SparkFun" deviceset="GND" device=""/>
@@
 </part>
 <part name="C33" library="rcl" deviceset="CPOL-EU" device="C/6032-28R" value="47uF/16V"/>
+<part name="L1" library="SparkFun" deviceset="INDUCTOR" device="CR75"/>
 </parts>
 <sheets>
@@
 <instance part="GND58" gate="1" x="25.4" y="-15.24"/>
 <instance part="GND59" gate="1" x="104.14" y="-27.94"/>
-<instance part="U$100" gate="G$1" x="81.28" y="27.94" rot="R90"/>
 <instance part="D100" gate="G$1" x="68.58" y="20.32" rot="R90"/>
 <instance part="GND60" gate="1" x="93.98" y="-5.08"/>
@@
 <instance part="TP81" gate="G$1" x="68.58" y="7.62"/>
 <instance part="C33" gate="G$1" x="114.3" y="20.32"/>
+<instance part="L1" gate="G$1" x="81.28" y="27.94" rot="R90"/>
 </instances>
 <busses>
@@
 <label x="111.76" y="27.94" size="1.778" layer="95"/>
 <pinref part="R37" gate="G$1" pin="1"/>
-<pinref part="U$100" gate="G$1" pin="2"/>
 <pinref part="5V" gate="G$1" pin="1"/>
 <pinref part="TP55" gate="G$1" pin="TP"/>
@@
 <wire x1="114.3" y1="22.86" x2="114.3" y2="27.94" width="0.1524" layer="91"/>
 <junction x="114.3" y="27.94"/>
+<pinref part="L1" gate="G$1" pin="2"/>
 </segment>
 </net>
@@
 <junction x="53.34" y="27.94"/>
 <pinref part="D100" gate="G$1" pin="C"/>
-<pinref part="U$100" gate="G$1" pin="1"/>
 <pinref part="U$3" gate="G$1" pin="PH"/>
 <pinref part="C15" gate="G$1" pin="1"/>
 <pinref part="TP54" gate="G$1" pin="TP"/>
+<pinref part="L1" gate="G$1" pin="1"/>
 </segment>
 </net>
@@
 </segment>
 </net>
-<net name="N$57" class="0">
+<net name="N$57" class="1">
 <segment>
 <wire x1="68.58" y1="129.54" x2="76.2" y2="129.54" width="0.1524" layer="91"/>
@@
 </segment>
 </net>
-<net name="12V5" class="0">
+<net name="12V5" class="1">
 <segment>
 <wire x1="83.82" y1="129.54" x2="88.9" y2="129.54" width="0.1524" layer="91"/>
@@
 </segment>
 </net>
-<net name="12V5VIN" class="2">
+<net name="12V5VIN" class="1">
 <segment>
 <wire x1="50.8" y1="111.76" x2="50.8" y2="114.3" width="0.1524" layer="91"/>
